File: pcbs/pico-sp0256/pico-sp0256.kicad_pcb (KiCad board)
At the start: 2 copper layers, 18.4 x 37.3 mm, 25 parts, among them J1 USB_B_Micro, J2 Conn_01x03_Female, U1 SP0256AL2, U2 W25Q128JVS, U3 NCP1117-3.3_SOT223, U5 RP2040, Y1 ABLS-12.000MHZ-B4-T

Commit message: Updates
Routing:
- net GND: track 0.00 -> 28.0 mm, vias 0 -> 8
- net SP_A4: track 0.00 -> 23.9 mm, vias 0 -> 1
- net SP_A3: track 0.00 -> 19.6 mm, vias 0 -> 1
- net QSPI_SD1: track 0.00 -> 17.8 mm, vias 0 -> 2
- net QSPI_SD3: track 0.00 -> 16.0 mm, vias 0 -> 2
- net QSPI_SS: track 0.00 -> 16.0 mm, vias 0 -> 2
- net SP_A2: track 0.00 -> 15.9 mm
- net SP_A1: track 0.00 -> 15.5 mm, vias 0 -> 2
- net QSPI_SCLK: track 0.00 -> 15.4 mm, vias 0 -> 2
- net QSPI_SD0: track 0.00 -> 14.0 mm, vias 0 -> 2
- net +3V3: track 0.00 -> 11.6 mm, vias 0 -> 7
- net QSPI_SD2: track 0.00 -> 11.3 mm
- net Net-(J1-Pad3): track 0.00 -> 8.77 mm
- net Net-(J1-Pad2): track 0.00 -> 8.66 mm
- net +1V1: track 0.00 -> 4.40 mm, vias 0 -> 2
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- added copper zone on In2.Cu, net +3V3
- added copper zone on In1.Cu, net GND
Other:
- copper layers 2 -> 4

Commit message: Updates
Parts:
- moved C12 1.28 mm to (76.7, 82.0), turned to 90 degrees
Routing:
- net SWCLK: track 0.00 -> 30.2 mm, vias 0 -> 3
- net SP_A5: track 0.00 -> 29.2 mm, vias 0 -> 2
- net SP_A6: track 0.00 -> 28.9 mm, vias 0 -> 2
- net SP_RESET_N: track 0.00 -> 28.6 mm, vias 0 -> 3
- net SP_A7: track 0.00 -> 24.6 mm, vias 0 -> 3
- net SP_A8: track 0.00 -> 21.1 mm, vias 0 -> 3
- net SP_LRQ_N: track 0.00 -> 20.2 mm, vias 0 -> 1
- net SP_SBY: track 0.00 -> 18.1 mm, vias 0 -> 2
- net VDD: track 0.00 -> 17.1 mm
- net GND: track 28.0 -> 43.4 mm, vias 8 -> 15
- net SWD: track 0.00 -> 14.9 mm, vias 0 -> 1
- net SP_ALD: track 0.00 -> 13.1 mm, vias 0 -> 2
- net SP_SE: track 0.00 -> 13.0 mm, vias 0 -> 1
- net Net-(D1-Pad1): track 0.00 -> 11.1 mm, vias 0 -> 2
- net SP_SBY_RES_N: track 0.00 -> 10.4 mm, vias 0 -> 2
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
Commit message: Updates
Parts:
- moved C7 3.06 mm to (80.5, 81.9), turned to 270 degrees
- moved C9 0.65 mm to (83.6, 79.1)
Routing:
- net +3V3: track 18.8 -> 28.7 mm, vias 10 -> 14
- net +1V1: track 8.52 -> 14.3 mm
- net GND: track 43.4 -> 44.9 mm, vias 15 -> 16
- net Net-(C2-Pad1): track 4.70 -> 5.57 mm
- net SP_SBY: track 18.1 -> 18.7 mm
Other:
- board text added: "SP0256 Emulator V1.0 Aug 2023 menadue@gmail.com"
